Commit message: urdf integration on progress

File: rise_assembler_model/urdf/irb120.xacro (robot description, xacro)
@@ -234,27 +234,9 @@
             <origin rpy="0 0 0" xyz="0 0 0"/>
         </joint>
-        <!-- Description of gripper -->
-        <link name="${prefix}gripper">
-            <visual>
-                <origin xyz="0 0 0" rpy="-1.57079632679 0 1.57079632679" />
-                <geometry>
-                    <mesh filename="package://irb120_description/meshes/visual/EndEffector.SLDPRT.STL" />
-                </geometry>
-                <material name="">
-                    <color rgba="1 1 1 1" />
-                </material>
-            </visual>
-            <collision>
-                <origin xyz="0 0 0" rpy="-1.57079632679 0 1.57079632679" />
-                <geometry>
-                    <mesh filename="package://irb120_description/meshes/collision/EndEffector.SLDPRT.STL" />
-                </geometry>
-            </collision>
-            <inertial>
-                <origin xyz="0 0 0" rpy="-1.57079632679 0 1.57079632679" />
-                <mass value="0.01"/>
-                <inertia ixx="1e-08" ixy="0" ixz="0" iyy="1e-08" iyz="0" izz="1e-08"/>
-            </inertial>
-        </link>
+        <!-- Description of the gripper -->
+        <!-- Call the model given from ROBOTIQ -->
+        <xacro:include filename="$(find robotiq_arg2f_model_visualization)/urdf/robotiq_arg2f_140_model_macro.xacro" />
+        <xacro:robotiq_arg2f_140 prefix=""/>
+        <!-- Robot kinetics parts -->
         <transmission name="${prefix}tran1">
             <type>transmission_interface/SimpleTransmission</type>

File: rise_assembler_model/urdf/robotiq_arg2f.xacro (robot description, xacro)
@@ -1,38 +1,38 @@
 <?xml version="1.0"?>
 <robot xmlns:xacro="http://ros.org/wiki/xacro">
-  <xacro:macro name="robotiq_arg2f_base_link" params="prefix">
-    <link name="${prefix}robotiq_arg2f_base_link">
-      <inertial>
-        <origin xyz="8.625E-08 -4.6583E-06 0.03145" rpy="0 0 0" />
-        <mass value="0.22652" />
-        <inertia ixx="0.00020005" ixy="-4.2442E-10" ixz="-2.9069E-10" iyy="0.00017832" iyz="-3.4402E-08" izz="0.00013478" />
-      </inertial>
-      <visual>
-        <origin xyz="0 0 0" rpy="0 0 0" />
-        <geometry>
-          <mesh filename="package://robotiq_arg2f_model_visualization/meshes/robotiq_arg2f_base_link_fine.stl" />
-        </geometry>
-        <material name="">
-          <color rgba="0.1 0.1 0.1 1" />
-        </material>
-      </visual>
-      <collision>
-        <origin xyz="0 0 0" rpy="0 0 ${pi / 2}" />
-        <geometry>
-          <mesh filename="package://robotiq_arg2f_model_visualization/meshes/robotiq_arg2f_base_link_coarse.stl" />
-        </geometry>
-      </collision>
-    </link>
-  </xacro:macro>
-  <xacro:macro name="finger_joints" params="prefix fingerprefix reflect">
-    <xacro:outer_finger_joint prefix="${prefix}" fingerprefix="${fingerprefix}"/>
-    <xacro:inner_knuckle_joint prefix="${prefix}" fingerprefix="${fingerprefix}" reflect="${reflect}"/>
-    <xacro:inner_finger_joint prefix="${prefix}" fingerprefix="${fingerprefix}"/>
-  </xacro:macro>
-  <xacro:macro name="finger_links" params="prefix fingerprefix stroke">
-    <xacro:outer_knuckle prefix="${prefix}" fingerprefix="${fingerprefix}" stroke="${stroke}"/>
-    <xacro:outer_finger prefix="${prefix}" fingerprefix="${fingerprefix}" stroke="${stroke}"/>
-    <xacro:inner_finger prefix="${prefix}" fingerprefix="${fingerprefix}" stroke="${stroke}"/>
-    <xacro:inner_knuckle prefix="${prefix}" fingerprefix="${fingerprefix}" stroke="${stroke}"/>
-  </xacro:macro>
+    <xacro:macro name="robotiq_arg2f_base_link" params="prefix">
+        <link name="${prefix}robotiq_arg2f_base_link">
+            <inertial>
+                <origin xyz="8.625E-08 -4.6583E-06 0.03145" rpy="0 0 0" />
+                <mass value="0.22652" />
+                <inertia ixx="0.00020005" ixy="-4.2442E-10" ixz="-2.9069E-10" iyy="0.00017832" iyz="-3.4402E-08" izz="0.00013478" />
+            </inertial>
+            <visual>
+                <origin xyz="0 0 0" rpy="0 0 0" />
+                <geometry>
+                    <mesh filename="package://robotiq_arg2f_model_visualization/meshes/robotiq_arg2f_base_link_fine.stl" />
+                </geometry>
+                <material name="">
+                    <color rgba="0.1 0.1 0.1 1" />
+                </material>
+            </visual>
+            <collision>
+                <origin xyz="0 0 0" rpy="0 0 ${pi / 2}" />
+                <geometry>
+                    <mesh filename="package://robotiq_arg2f_model_visualization/meshes/robotiq_arg2f_base_link_coarse.stl" />
+                </geometry>
+            </collision>
+        </link>
+    </xacro:macro>
+    <xacro:macro name="finger_joints" params="prefix fingerprefix reflect">
+        <xacro:outer_finger_joint prefix="${prefix}" fingerprefix="${fingerprefix}"/>
+        <xacro:inner_knuckle_joint prefix="${prefix}" fingerprefix="${fingerprefix}" reflect="${reflect}"/>
+        <xacro:inner_finger_joint prefix="${prefix}" fingerprefix="${fingerprefix}"/>
+    </xacro:macro>
+    <xacro:macro name="finger_links" params="prefix fingerprefix stroke">
+        <xacro:outer_knuckle prefix="${prefix}" fingerprefix="${fingerprefix}" stroke="${stroke}"/>
+        <xacro:outer_finger prefix="${prefix}" fingerprefix="${fingerprefix}" stroke="${stroke}"/>
+        <xacro:inner_finger prefix="${prefix}" fingerprefix="${fingerprefix}" stroke="${stroke}"/>
+        <xacro:inner_knuckle prefix="${prefix}" fingerprefix="${fingerprefix}" stroke="${stroke}"/>
+    </xacro:macro>
 </robot>
