Commit message: starting task planning

File: rise_assembler_model/urdf/robotiq_arg2f.xacro (robot description, xacro)
@@ -11,5 +11,5 @@
                 <origin xyz="0 0 0" rpy="0 0 0" />
                 <geometry>
-                    <mesh filename="package://robotiq_arg2f_model_visualization/meshes/robotiq_arg2f_base_link_fine.stl" />
+                    <mesh filename="$(find rise_assembler_model)/mesh/gripper/robotiq_arg2f_base_link_fine.stl" />
                 </geometry>
                 <material name="">
@@ -20,5 +20,5 @@
                 <origin xyz="0 0 0" rpy="0 0 ${pi / 2}" />
                 <geometry>
-                    <mesh filename="package://robotiq_arg2f_model_visualization/meshes/robotiq_arg2f_base_link_coarse.stl" />
+                    <mesh filename="$(find rise_assembler_model)/mesh/gripper/robotiq_arg2f_base_link_coarse.stl" />
                 </geometry>
             </collision>

File: rise_assembler_model/urdf/robotiq_arg2f_140_model.xacro (robot description, xacro)
@@ -1,5 +1,5 @@
 <?xml version="1.0"?>
 <robot name="robotiq_arg2f_140_model" xmlns:xacro="http://ros.org/wiki/xacro">
-  <xacro:include filename="$(find robotiq_arg2f_model_visualization)/urdf/robotiq_arg2f_140_model_macro.xacro" />
+  <xacro:include filename="$(find rise_assembler_model)/urdf/robotiq_arg2f_140_model_macro.xacro" />
   <xacro:robotiq_arg2f_140 prefix=""/>
 </robot>

File: rise_assembler_model/urdf/robotiq_arg2f_140_model_macro.xacro (robot description, xacro)
@@ -12,5 +12,5 @@
                 <origin xyz="0 0 0" rpy="0 0 0" />
                 <geometry>
-                    <mesh filename="package://robotiq_arg2f_model_visualization/meshes/robotiq_arg2f_${stroke}_outer_knuckle.stl" />
+                    <mesh filename="$(find rise_assembler_model)/mesh/gripper/robotiq_arg2f_${stroke}_outer_knuckle.stl" />
                 </geometry>
                 <material name="">
@@ -21,5 +21,5 @@
                 <origin xyz="0 0 0" rpy="0 0 0" />
                 <geometry>
-                    <mesh filename="package://robotiq_arg2f_model_visualization/meshes/robotiq_arg2f_${stroke}_outer_knuckle.stl" />
+                    <mesh filename="$(find rise_assembler_model)/mesh/gripper/robotiq_arg2f_${stroke}_outer_knuckle.stl" />
                 </geometry>
             </collision>
@@ -36,5 +36,5 @@
                 <origin xyz="0 0 0" rpy="0 0 0" />
                 <geometry>
-                    <mesh filename="package://robotiq_arg2f_model_visualization/meshes/robotiq_arg2f_${stroke}_outer_finger.stl" />
+                    <mesh filename="$(find rise_assembler_model)/mesh/gripper/robotiq_arg2f_${stroke}_outer_finger.stl" />
                 </geometry>
                 <material name="">
@@ -45,5 +45,5 @@
                 <origin xyz="0 0 0" rpy="0 0 0" />
                 <geometry>
-                    <mesh filename="package://robotiq_arg2f_model_visualization/meshes/robotiq_arg2f_${stroke}_outer_finger.stl" />
+                    <mesh filename="$(find rise_assembler_model)/mesh/gripper/robotiq_arg2f_${stroke}_outer_finger.stl" />
                 </geometry>
             </collision>
@@ -60,5 +60,5 @@
                 <origin xyz="0 0 0" rpy="0 0 0" />
                 <geometry>
-                    <mesh filename="package://robotiq_arg2f_model_visualization/meshes/robotiq_arg2f_${stroke}_inner_knuckle.stl" />
+                    <mesh filename="$(find rise_assembler_model)/mesh/gripper/robotiq_arg2f_${stroke}_inner_knuckle.stl" />
                 </geometry>
                 <material name="">
@@ -69,5 +69,5 @@
                 <origin xyz="0 0 0" rpy="0 0 0" />
                 <geometry>
-                    <mesh filename="package://robotiq_arg2f_model_visualization/meshes/robotiq_arg2f_${stroke}_inner_knuckle.stl" />
+                    <mesh filename="$(find rise_assembler_model)/mesh/gripper/robotiq_arg2f_${stroke}_inner_knuckle.stl" />
                 </geometry>
             </collision>
@@ -84,5 +84,5 @@
                 <origin xyz="0 0 0" rpy="0 0 0" />
                 <geometry>
-                    <mesh filename="package://robotiq_arg2f_model_visualization/meshes/robotiq_arg2f_${stroke}_inner_finger.stl" />
+                    <mesh filename="$(find rise_assembler_model)/mesh/gripper/robotiq_arg2f_${stroke}_inner_finger.stl" />
                 </geometry>
                 <material name="">
@@ -93,5 +93,5 @@
                 <origin xyz="0 0 0" rpy="0 0 0" />
                 <geometry>
-                    <mesh filename="package://robotiq_arg2f_model_visualization/meshes/robotiq_arg2f_${stroke}_inner_finger.stl" />
+                    <mesh filename="$(find rise_assembler_model)/mesh/gripper/robotiq_arg2f_${stroke}_inner_finger.stl" />
                 </geometry>
             </collision>
@@ -126,5 +126,5 @@
         </joint>
     </xacro:macro>
-    <xacro:include filename="$(find robotiq_arg2f_model_visualization)/urdf/robotiq_arg2f.xacro" />
+    <xacro:include filename="$(find rise_assembler_model)/urdf/robotiq_arg2f.xacro" />
     <xacro:macro name="finger_joint" params="prefix">
         <joint name="${prefix}finger_joint" type="revolute">
