Commit message: code applied in video: pick-up four pins

File: rise_assembler_model/urdf/rise_assembler.2.xacro (robot description, xacro)
@@ -18,5 +18,5 @@
         <parent link="world"/>
         <child link="${irb120_ns}base_link"/>
-        <origin rpy="0 0 0" xyz="0 0 0.76"/>
+        <origin rpy="0 0 0" xyz="0 0 0"/>
     </joint>
     <!-- Description of IRB120 robot -->
@@ -80,5 +80,5 @@
         <child link="${irb120_ns}link_2"/>
         <limit effort="20" lower="-1.91986" upper="1.91986" velocity="4.36332"/>
-        <axis xyz="0 -1 0"/>
+        <axis xyz="0 1 0"/>
         <dynamics damping="1" friction="0"/>
     </joint>
@@ -111,5 +111,5 @@
         <child link="${irb120_ns}link_3"/>
         <limit effort="20" lower="-1.91986" upper="1.22173" velocity="4.36332"/>
-        <axis xyz="0 -1 0"/>
+        <axis xyz="0 1 0"/>
         <dynamics damping="1" friction="0.0"/>
     </joint>
@@ -173,5 +173,5 @@
         <child link="${irb120_ns}link_5"/>
         <limit effort="20" lower="-2.094395" upper="2.094395" velocity="5.58505"/>
-        <axis xyz="0 -1 0"/>
+        <axis xyz="0 1 0"/>
         <dynamics damping="1" friction="0.0"/>
     </joint>

File: rise_assembler_model/urdf/rise_assembler.xacro (robot description, xacro)
@@ -11,4 +11,6 @@
         </plugin>
     </gazebo>
+    <xacro:property name="irb120_ns" value="" />
+    <xacro:property name="gripper_ns" value="" />
     <!-- Used for fixing robot to Gazebo 'base_link' -->
     <link name="world"/>
@@ -16,8 +18,6 @@
         <parent link="world"/>
         <child link="${irb120_ns}base_link"/>
-        <origin rpy="0 0 0" xyz="0 0 0.76"/>
-    </joint>
-    <xacro:property name="irb120_ns" value="" />
-    <xacro:property name="gripper_ns" value="" />
+        <origin rpy="0 0 0" xyz="0 0 0"/>
+    </joint>
     <!-- Description of IRB120 robot -->
     <!-- Description of base_link -->
@@ -31,12 +31,12 @@
             <origin xyz="0 0 0" rpy="0 0 0"/>
             <geometry>
-                <mesh filename="$(find rise_assembler_model)/mesh/irb120/base_link.stl"/>
-            </geometry>
-            <xacro:material_abb_orange />
-        </visual>
-        <collision>
-            <origin xyz="0 0 0" rpy="0 0 0"/>
-            <geometry>
-                <mesh filename="$(find rise_assembler_model)/collision/irb120/base_link.stl"/>
+                <mesh filename="package://rise_assembler_model/mesh/irb120/base_link.stl"/>
+            </geometry>
+            <xacro:material_abb_orange />
+        </visual>
+        <collision>
+            <origin xyz="0 0 0" rpy="0 0 0"/>
+            <geometry>
+                <mesh filename="package://rise_assembler_model/collision/irb120/base_link.stl"/>
             </geometry>
             <xacro:material_abb_yellow />
@@ -62,12 +62,12 @@
             <origin xyz="0 0 0" rpy="0 0 0"/>
             <geometry>
-                <mesh filename="$(find rise_assembler_model)/mesh/irb120/link_1.stl"/>
-            </geometry>
-            <xacro:material_abb_orange />
-        </visual>
-        <collision>
-            <origin xyz="0 0 0" rpy="0 0 0"/>
-            <geometry>
-                <mesh filename="$(find rise_assembler_model)/collision/irb120/link_1.stl"/>
+                <mesh filename="package://rise_assembler_model/mesh/irb120/link_1.stl"/>
+            </geometry>
+            <xacro:material_abb_orange />
+        </visual>
+        <collision>
+            <origin xyz="0 0 0" rpy="0 0 0"/>
+            <geometry>
+                <mesh filename="package://rise_assembler_model/collision/irb120/link_1.stl"/>
             </geometry>
             <xacro:material_abb_yellow />
@@ -80,5 +80,5 @@
         <child link="${irb120_ns}link_2"/>
         <limit effort="20" lower="-1.91986" upper="1.91986" velocity="4.36332"/>
-        <axis xyz="0 -1 0"/>
+        <axis xyz="0 1 0"/>
         <dynamics damping="1" friction="0"/>
     </joint>
@@ -93,12 +93,12 @@
             <origin xyz="0 0 0" rpy="0 0 0"/>
             <geometry>
-                <mesh filename="$(find rise_assembler_model)/mesh/irb120/link_2.stl"/>
-            </geometry>
-            <xacro:material_abb_orange />
-        </visual>
-        <collision>
-            <origin xyz="0 0 0" rpy="0 0 0"/>
-            <geometry>
-                <mesh filename="$(find rise_assembler_model)/collision/irb120/link_2.stl"/>
+                <mesh filename="package://rise_assembler_model/mesh/irb120/link_2.stl"/>
+            </geometry>
+            <xacro:material_abb_orange />
+        </visual>
+        <collision>
+            <origin xyz="0 0 0" rpy="0 0 0"/>
+            <geometry>
+                <mesh filename="package://rise_assembler_model/collision/irb120/link_2.stl"/>
             </geometry>
             <xacro:material_abb_yellow />
@@ -111,5 +111,5 @@
         <child link="${irb120_ns}link_3"/>
         <limit effort="20" lower="-1.91986" upper="1.22173" velocity="4.36332"/>
-        <axis xyz="0 -1 0"/>
+        <axis xyz="0 1 0"/>
         <dynamics damping="1" friction="0.0"/>
     </joint>
@@ -124,12 +124,12 @@
             <origin xyz="0 0 0" rpy="0 0 0"/>
             <geometry>
-                <mesh filename="$(find rise_assembler_model)/mesh/irb120/link_3.stl"/>
-            </geometry>
-            <xacro:material_abb_orange />
-        </visual>
-        <collision>
-            <origin xyz="0 0 0" rpy="0 0 0"/>
-            <geometry>
-                <mesh filename="$(find rise_assembler_model)/collision/irb120/link_3.stl"/>
+                <mesh filename="package://rise_assembler_model/mesh/irb120/link_3.stl"/>
+            </geometry>
+            <xacro:material_abb_orange />
+        </visual>
+        <collision>
+            <origin xyz="0 0 0" rpy="0 0 0"/>
+            <geometry>
+                <mesh filename="package://rise_assembler_model/collision/irb120/link_3.stl"/>
             </geometry>
             <xacro:material_abb_yellow />
@@ -141,6 +141,6 @@
         <parent link="${irb120_ns}link_3"/>
         <child link="${irb120_ns}link_4"/>
-        <limit effort="20" lower="-4" upper="4" velocity="5.58505"/>
-        <axis xyz="1 0 0"/>
+        <limit effort="20" lower="-2.792526" upper="2.792526" velocity="5.58505"/>
+        <axis xyz="-1 0 0"/>
         <dynamics damping="1" friction="0"/>
     </joint>
@@ -155,12 +155,12 @@
             <origin xyz="0 0 0" rpy="0 0 0"/>
             <geometry>
-                <mesh filename="$(find rise_assembler_model)/mesh/irb120/link_4.stl"/>
-            </geometry>
-            <xacro:material_abb_orange />
-        </visual>
-        <collision>
-            <origin xyz="0 0 0" rpy="0 0 0"/>
-            <geometry>
-                <mesh filename="$(find rise_assembler_model)/collision/irb120/link_4.stl"/>
+                <mesh filename="package://rise_assembler_model/mesh/irb120/link_4.stl"/>
+            </geometry>
+            <xacro:material_abb_orange />
+        </visual>
+        <collision>
+            <origin xyz="0 0 0" rpy="0 0 0"/>
+            <geometry>
+                <mesh filename="package://rise_assembler_model/collision/irb120/link_4.stl"/>
             </geometry>
             <xacro:material_abb_yellow />
@@ -173,5 +173,5 @@
         <child link="${irb120_ns}link_5"/>
         <limit effort="20" lower="-2.094395" upper="2.094395" velocity="5.58505"/>
-        <axis xyz="0 -1 0"/>
+        <axis xyz="0 1 0"/>
         <dynamics damping="1" friction="0.0"/>
     </joint>
@@ -186,12 +186,12 @@
             <origin xyz="0 0 0" rpy="0 0 0"/>
             <geometry>
-                <mesh filename="$(find rise_assembler_model)/mesh/irb120/link_5.stl"/>
-            </geometry>
-            <xacro:material_abb_orange />
-        </visual>
-        <collision>
-            <origin xyz="0 0 0" rpy="0 0 0"/>
-            <geometry>
-                <mesh filename="$(find rise_assembler_model)/collision/irb120/link_5.stl"/>
+                <mesh filename="package://rise_assembler_model/mesh/irb120/link_5.stl"/>
+            </geometry>
+            <xacro:material_abb_orange />
+        </visual>
+        <collision>
+            <origin xyz="0 0 0" rpy="0 0 0"/>
+            <geometry>
+                <mesh filename="package://rise_assembler_model/collision/irb120/link_5.stl"/>
             </geometry>
             <xacro:material_abb_yellow />
@@ -203,5 +203,5 @@
         <parent link="${irb120_ns}link_5"/>
         <child link="${irb120_ns}link_6"/>
-        <limit effort="20" lower="-4" upper="4" velocity="7.33038"/>
+        <limit effort="20" lower="-6.981317" upper="6.981317" velocity="7.33038"/>
         <axis xyz="1 0 0"/>
         <dynamics damping="1" friction="0.0"/>
@@ -217,5 +217,5 @@
             <origin xyz="0 0 0" rpy="0 0 0"/>
             <geometry>
-                <mesh filename="$(find rise_assembler_model)/mesh/irb120/link_6.stl"/>
+                <mesh filename="package://rise_assembler_model/mesh/irb120/link_6.stl"/>
             </geometry>
             <xacro:material_abb_black />
@@ -224,5 +224,5 @@
             <origin xyz="0 0 0" rpy="0 0 0"/>
             <geometry>
-                <mesh filename="$(find rise_assembler_model)/collision/irb120/link_6.stl"/>
+                <mesh filename="package://rise_assembler_model/collision/irb120/link_6.stl"/>
             </geometry>
             <xacro:material_abb_yellow />

File: rise_assembler_model/urdf/robotiq_arg2f.xacro (robot description, xacro)
@@ -11,5 +11,5 @@
                 <origin xyz="0 0 0" rpy="0 0 0" />
                 <geometry>
-                    <mesh filename="$(find rise_assembler_model)/mesh/gripper/robotiq_arg2f_base_link_fine.stl" />
+                    <mesh filename="package://rise_assembler_model/mesh/gripper/robotiq_arg2f_base_link_fine.stl" />
                 </geometry>
                 <material name="">
@@ -20,5 +20,5 @@
                 <origin xyz="0 0 0" rpy="0 0 ${pi / 2}" />
                 <geometry>
-                    <mesh filename="$(find rise_assembler_model)/mesh/gripper/robotiq_arg2f_base_link_coarse.stl" />
+                    <mesh filename="package://rise_assembler_model/mesh/gripper/robotiq_arg2f_base_link_coarse.stl" />
                 </geometry>
             </collision>

File: rise_assembler_model/urdf/robotiq_arg2f_140_model_macro.xacro (robot description, xacro)
@@ -12,5 +12,5 @@
                 <origin xyz="0 0 0" rpy="0 0 0" />
                 <geometry>
-                    <mesh filename="$(find rise_assembler_model)/mesh/gripper/robotiq_arg2f_${stroke}_outer_knuckle.stl" />
+                    <mesh filename="package://rise_assembler_model/mesh/gripper/robotiq_arg2f_${stroke}_outer_knuckle.stl" />
                 </geometry>
                 <material name="">
@@ -21,5 +21,5 @@
                 <origin xyz="0 0 0" rpy="0 0 0" />
                 <geometry>
-                    <mesh filename="$(find rise_assembler_model)/mesh/gripper/robotiq_arg2f_${stroke}_outer_knuckle.stl" />
+                    <mesh filename="package://rise_assembler_model/mesh/gripper/robotiq_arg2f_${stroke}_outer_knuckle.stl" />
                 </geometry>
             </collision>
@@ -36,5 +36,5 @@
                 <origin xyz="0 0 0" rpy="0 0 0" />
                 <geometry>
-                    <mesh filename="$(find rise_assembler_model)/mesh/gripper/robotiq_arg2f_${stroke}_outer_finger.stl" />
+                    <mesh filename="package://rise_assembler_model/mesh/gripper/robotiq_arg2f_${stroke}_outer_finger.stl" />
                 </geometry>
                 <material name="">
@@ -45,5 +45,5 @@
                 <origin xyz="0 0 0" rpy="0 0 0" />
                 <geometry>
-                    <mesh filename="$(find rise_assembler_model)/mesh/gripper/robotiq_arg2f_${stroke}_outer_finger.stl" />
+                    <mesh filename="package://rise_assembler_model/mesh/gripper/robotiq_arg2f_${stroke}_outer_finger.stl" />
                 </geometry>
             </collision>
@@ -60,5 +60,5 @@
                 <origin xyz="0 0 0" rpy="0 0 0" />
                 <geometry>
-                    <mesh filename="$(find rise_assembler_model)/mesh/gripper/robotiq_arg2f_${stroke}_inner_knuckle.stl" />
+                    <mesh filename="package://rise_assembler_model/mesh/gripper/robotiq_arg2f_${stroke}_inner_knuckle.stl" />
                 </geometry>
                 <material name="">
@@ -69,5 +69,5 @@
                 <origin xyz="0 0 0" rpy="0 0 0" />
                 <geometry>
-                    <mesh filename="$(find rise_assembler_model)/mesh/gripper/robotiq_arg2f_${stroke}_inner_knuckle.stl" />
+                    <mesh filename="package://rise_assembler_model/mesh/gripper/robotiq_arg2f_${stroke}_inner_knuckle.stl" />
                 </geometry>
             </collision>
@@ -84,5 +84,5 @@
                 <origin xyz="0 0 0" rpy="0 0 0" />
                 <geometry>
-                    <mesh filename="$(find rise_assembler_model)/mesh/gripper/robotiq_arg2f_${stroke}_inner_finger.stl" />
+                    <mesh filename="package://rise_assembler_model/mesh/gripper/robotiq_arg2f_${stroke}_inner_finger.stl" />
                 </geometry>
                 <material name="">
@@ -93,5 +93,5 @@
                 <origin xyz="0 0 0" rpy="0 0 0" />
                 <geometry>
-                    <mesh filename="$(find rise_assembler_model)/mesh/gripper/robotiq_arg2f_${stroke}_inner_finger.stl" />
+                    <mesh filename="package://rise_assembler_model/mesh/gripper/robotiq_arg2f_${stroke}_inner_finger.stl" />
                 </geometry>
             </collision>
