Commit message: successed to translate straight rods

File: rise_assembler_model/urdf/rise_assembler.xacro (robot description, xacro)
@@ -142,5 +142,5 @@
         <child link="${irb120_ns}link_4"/>
         <limit effort="20" lower="-2.792526" upper="2.792526" velocity="5.58505"/>
-        <axis xyz="-1 0 0"/>
+        <axis xyz="1 0 0"/>
         <dynamics damping="1" friction="0"/>
     </joint>
