Commit message: added manual controller and gui sketch

File: rise_assembler_model/urdf/rise_assembler_backup.xacro (robot description, xacro)
@@ -18,5 +18,5 @@
         <parent link="world"/>
         <child link="${irb120_ns}base_link"/>
-        <origin rpy="0 0 0" xyz="0 0 0.76"/>
+        <origin rpy="0 0 0" xyz="0 0 0"/>
     </joint>
     <!-- Description of IRB120 robot -->
@@ -80,5 +80,5 @@
         <child link="${irb120_ns}link_2"/>
         <limit effort="20" lower="-1.91986" upper="1.91986" velocity="4.36332"/>
-        <axis xyz="0 -1 0"/>
+        <axis xyz="0 1 0"/>
         <dynamics damping="1" friction="0"/>
     </joint>
@@ -111,5 +111,5 @@
         <child link="${irb120_ns}link_3"/>
         <limit effort="20" lower="-1.91986" upper="1.22173" velocity="4.36332"/>
-        <axis xyz="0 -1 0"/>
+        <axis xyz="0 1 0"/>
         <dynamics damping="1" friction="0.0"/>
     </joint>
@@ -141,5 +141,5 @@
         <parent link="${irb120_ns}link_3"/>
         <child link="${irb120_ns}link_4"/>
-        <limit effort="20" lower="-4" upper="4" velocity="5.58505"/>
+        <limit effort="20" lower="-2.792526" upper="2.792526" velocity="5.58505"/>
         <axis xyz="1 0 0"/>
         <dynamics damping="1" friction="0"/>
@@ -173,5 +173,5 @@
         <child link="${irb120_ns}link_5"/>
         <limit effort="20" lower="-2.094395" upper="2.094395" velocity="5.58505"/>
-        <axis xyz="0 -1 0"/>
+        <axis xyz="0 1 0"/>
         <dynamics damping="1" friction="0.0"/>
     </joint>
@@ -203,5 +203,5 @@
         <parent link="${irb120_ns}link_5"/>
         <child link="${irb120_ns}link_6"/>
-        <limit effort="20" lower="-4" upper="4" velocity="7.33038"/>
+        <limit effort="20" lower="-6.981317" upper="6.981317" velocity="7.33038"/>
         <axis xyz="1 0 0"/>
         <dynamics damping="1" friction="0.0"/>
@@ -229,5 +229,5 @@
         </collision>
     </link>
-    <!-- Description of the gripper -->
+    Description of the gripper
     <xacro:include filename="$(find rise_assembler_model)/urdf/robotiq_arg2f_140_model.xacro" />
     <!-- bolting between link 6 and gripper -->
